Commit message: feat(herramienta): acople porta-bisturí en Gazebo, y el TCP pasa a la punta de la hoja
El efector deja de ser un frame virtual: el acople del CAD se monta en tool0 con
malla, colisiones y masa, y gripper_tcp pasa de 0.141 m (TCP del gripper Robotiq,
que ya no se monta) a 0.162686 m, que es la punta de la hoja.

Geometría, deducida de la malla y no supuesta:

- Origen del OBJ == tool0. El acople tiene un rebaje Ø63.4 mm cuyo fondo es una
  cara plana exactamente en z=0 (anillo r=5.550..31.700 mm); como el rebaje mide
  7.0 mm y el resalte de la brida 6.5, hace tope contra la cara de la brida.
- Punta de la hoja: vértice de z máximo, (0.316, 4.280, 162.686) mm.
- Filo hacia -Y del acople (bisel trazado a media altura del espesor de 0.4 mm),
  igual que el conector de herramienta del UR5e (protuberancia de wrist3.dae a
  radio 43.5 mm, azimut -90 deg). Montaje con rotación identidad => el filo
  apunta a la rosca de conexión, como pedía la referencia.
- Con tcp_orientation_rpy=[pi,0,pi] el eje Y de la herramienta es el +Y de
  base_link y el trazo recorre Y con cut_direction=-1: el filo va POR DELANTE
  del movimiento y la hoja corta en su propio plano.

Los 171.686 mm de mounting_measurements.png menos los 6.5 del resalte darían
165.186. Se adopta 162.686 porque el datum de esa cota cae 9.0 mm por detrás de
tool0, no 6.5 (medido: la flecha queda 2.0 mm por detrás de la cara trasera del
acople, que está en z=-7), y porque la cota de la malla no depende de la altura
del resalte. Anotado en docs/00_assumptions.md con cómo revertirlo.

A1 LEVANTADO: 0.182 kg, CoG y tensor de inercia del CAD entran a la vez en la
planta (scalpel_tool.xacro) y en el modelo de Pinocchio (tool_mass/tool_com/
tool_inertia en los seis YAML). Van emparejados o el controlador compensaría una
gravedad que no es la de la planta.

Colisiones con 5 primitivas, no con la malla: un trimesh de 70904 caras hunde el
RTF (ya medido en este workspace con la mesa de cirugía).

Verificado en Gazebo:
- gravity_comp, 28 s de sostén en q_init: error 0.000000 rad en las 6 juntas.
- Incisión completa (14642 muestras): TRACK -> HOLD_END -> DONE sin abortos,
  seguimiento RMS 0.023 mm / máx 0.187 mm.
- Holgura de la punta sobre la surgery_table: 15.00 mm en toda la trayectoria,
  sin cambiar la altura del trazo. Con el offset viejo la punta habría bajado a
  -6.7 mm, o sea dentro de la mesa: la colisión venía del TCP, no del trazo.
- sigma_min(J) baja de 0.2168 a 0.1564 por el TCP más largo (umbral 0.05).

Las campañas de las FASES 2 y 5 se corrieron sin herramienta: siguen valiendo
para lo que medían, pero no son comparables con corridas nuevas.

De paso, A4 decía [pi,0,-pi/2] cuando los YAML llevan [pi,0,pi] desde 0ecb25c.

Co-Authored-By: Claude Opus 5 <noreply@anthropic.com>

File: ur5_dyn_control/urdf/ur5e_effort.urdf.xacro (robot description, xacro)
@@ -1,8 +1,9 @@
 <?xml version="1.0"?>
 <!--
-  UR5e arm only, con interfaz de comando EFFORT, para control por torque en
-  Gazebo Fortress / ROS 2 Humble. Sin gripper Robotiq, pero manteniendo el
-  frame 'gripper_tcp' a 0.141 m de tool0 (misma cadena que
-  ur5_robotiq_2f85.urdf.xacro — ver ur5_pick_place/urdf/ur5e.urdf.xacro).
+  UR5e con interfaz de comando EFFORT, para control por torque en Gazebo
+  Fortress / ROS 2 Humble. Sin gripper Robotiq: el efector es el ACOPLE
+  PORTA-BISTURI de la campana de incision (scalpel_tool.xacro), y el frame
+  'gripper_tcp' pasa a ser la punta de la hoja, a 0.162686 m de tool0
+  (antes 0.141 m, que era el TCP del gripper Robotiq).
   Diferencias respecto a ur5e.urdf.xacro de ur5_pick_place:
    - xacro:ur_robot se instancia con generate_ros2_control_tag="false"
@@ -30,4 +31,6 @@
   <xacro:include filename="$(find ur_description)/urdf/ur_macro.xacro"/>
   <xacro:include filename="$(find ur5_dyn_control)/urdf/ur5e_effort.ros2_control.xacro"/>
+  <!-- Define la property scalpel_tcp_offset_z y el macro ur5_scalpel_tool. -->
+  <xacro:include filename="$(find ur5_dyn_control)/urdf/scalpel_tool.xacro"/>
   <!-- ===== Properties ===== -->
   <xacro:property name="initial_positions_file" value="$(arg initial_positions_file)"/>
@@ -68,13 +71,23 @@
     </plugin>
   </gazebo>
+  <!-- ===== Acople porta-bisturi ===== -->
+  <!-- Origen y orientacion IDENTIDAD sobre tool0; el porque esta en la
+       cabecera de scalpel_tool.xacro (la malla apoya por el fondo de su
+       rebaje, que cae exactamente en z = 0 = cara de la brida). -->
+  <xacro:ur5_scalpel_tool parent="$(arg tf_prefix)tool0" prefix="$(arg tf_prefix)"/>
   <!-- ===== gripper_tcp frame ===== -->
-  <!-- Frame fijo a 0.141 m de tool0 en Z local (offset combinado adaptador +
-       gripper). Identico al gripper_tcp de ur5_robotiq_2f85.urdf.xacro:
-       mantiene la pose TCP del gripper aunque el modelo no lo lleve. -->
+  <!-- Ahora es la PUNTA DE LA HOJA: scalpel_tcp_offset_z = 0.162686 m de tool0
+       en Z local (antes 0.141 m, el offset del gripper Robotiq que ya no se
+       monta). El nombre se conserva porque es el frame que la IK de
+       ur5_kinematics resuelve POR NOMBRE (JointReferenceGenerator, IKWrapper);
+       renombrarlo obligaria a tocar ur5_kinematics y ur5_pick_place, fuera de
+       alcance.
+       Este valor y el `tcp_offset_z` de config/*.yaml TIENEN que coincidir:
+       es el supuesto A2 (docs/00_assumptions.md). -->
   <link name="gripper_tcp"/>
   <joint name="gripper_tcp_joint" type="fixed">
     <parent link="$(arg tf_prefix)tool0"/>
     <child  link="gripper_tcp"/>
-    <origin xyz="0 0 0.141" rpy="0 0 0"/>
+    <origin xyz="0 0 ${scalpel_tcp_offset_z}" rpy="0 0 0"/>
   </joint>
 </robot>
